Commit message: Adjusted gripper collision box

File: src/robot_description/urdf/adaptive_gripper.urdf.xacro (robot description, xacro)
@@ -37,7 +37,7 @@
       <collision>
         <geometry>
-          <box size="0.065 0.025 0.025"/>
-        </geometry>
-        <origin xyz="0.0 0.0 0.0" rpy="0 0 0"/>
+          <box size="0.065 0.025 0.052"/> // original 0.065 0.025 0.025
+        </geometry>
+        <origin xyz="0.0 0.0 0.013" rpy="0 0 0"/>
       </collision>
     </link>
