Commit message: Adjusted camera mount collision box

File: src/robot_description/urdf/mounted_d435i.urdf.xacro (robot description, xacro)
@@ -14,10 +14,4 @@
 				</material>
 			</visual>
-			<collision>
-				<origin xyz="0 0 ${-mount_collision_padding + (mount_collision_z + 2 * mount_collision_padding) / 2}" rpy="0 0 0" />
-				<geometry>
-					<box size="${mount_collision_x + 2 * mount_collision_padding} ${mount_collision_y + 2 * mount_collision_padding} ${mount_collision_z + 2 * mount_collision_padding}" />
-				</geometry>
-			</collision>
 		</link>
 		<joint name="camera_mount_base_joint" type="fixed">
@@ -26,5 +20,12 @@
 			<child link="camera_mount_base" />
 		</joint>
-		<link name="${name}_mount" />
+		<link name="${name}_mount">
+			<collision>
+				<origin xyz="0.006 0 ${-mount_collision_padding + (mount_collision_z + 2 * mount_collision_padding) / 2 - 0.0145}" rpy="0 0 0" />
+				<geometry>
+					<box size="${mount_collision_x + 2 * mount_collision_padding} ${mount_collision_y + 2 * mount_collision_padding} ${mount_collision_z + 2 * mount_collision_padding}" />
+				</geometry>
+			</collision>
+		</link>
 		<joint name="${name}_mount_top" type="fixed">
 			<parent link="camera_mount_base" />

Commit message: Adjusted d435i collision box

File: src/robot_description/urdf/mounted_d435i.urdf.xacro (robot description, xacro)
@@ -22,5 +22,5 @@
 		<link name="${name}_mount">
 			<collision>
-				<origin xyz="0.006 0 ${-mount_collision_padding + (mount_collision_z + 2 * mount_collision_padding) / 2 - 0.0145}" rpy="0 0 0" />
+				<origin xyz="0.006 0.005 ${-mount_collision_padding + (mount_collision_z + 2 * mount_collision_padding) / 2 - 0.0145}" rpy="0 0 0" />
 				<geometry>
 					<box size="${mount_collision_x + 2 * mount_collision_padding} ${mount_collision_y + 2 * mount_collision_padding} ${mount_collision_z + 2 * mount_collision_padding}" />
