Commit message: Fixed paths to camera meshe and URDF

File: src/robot_description/urdf/rgbd_camera/_d435.urdf.xacro (robot description, xacro)
@@ -66,5 +66,5 @@
           <origin xyz="${d435_zero_depth_to_glass + d435_glass_to_front} ${-d435_cam_depth_py} 0" rpy="${M_PI/2} 0 ${M_PI/2}"/>
           <geometry>
-            <mesh filename="package://robot_description/meshes/d435.dae" />
+            <mesh filename="package://robot_description/meshes/rgbd_camera/d435.dae" />
           </geometry>
         </xacro:if>

File: src/robot_description/urdf/rgbd_camera/mounted_d435i.urdf.xacro (robot description, xacro)
@@ -1,5 +1,5 @@
 <?xml version="1.0"?>
 <robot name="mounted_d435i" xmlns:xacro="http://www.ros.org/wiki/xacro">
-	<xacro:include filename="$(find robot_description)/urdf/_d435i.urdf.xacro"/>
+	<xacro:include filename="$(find robot_description)/urdf/rgbd_camera/_d435i.urdf.xacro"/>
 	<xacro:macro name="mounted_d435i" params="parent *origin name:=camera use_nominal_extrinsics:=false mount_mesh_scale:=1.0 mount_mesh_x:=0.04073 mount_mesh_y:=0.1082 mount_mesh_z:=0.05081 mount_collision_x:=0.04073 mount_collision_y:=0.1082 mount_collision_z:=0.05081">
 		<xacro:property name="mount_collision_padding" value="0.005" />

Commit message: Fixed rgbd camera so it shows in Gazebo

File: src/robot_description/urdf/rgbd_camera/_d435.urdf.xacro (robot description, xacro)
@@ -66,5 +66,5 @@
           <origin xyz="${d435_zero_depth_to_glass + d435_glass_to_front} ${-d435_cam_depth_py} 0" rpy="${M_PI/2} 0 ${M_PI/2}"/>
           <geometry>
-            <mesh filename="package://robot_description/meshes/rgbd_camera/d435.dae" />
+            <mesh filename="file://$(find robot_description)/meshes/rgbd_camera/d435.dae" />
           </geometry>
         </xacro:if>
