Commit message: Moved collisions to same link as visual

File: src/robot_description/urdf/rgbd_camera/mounted_d435i.urdf.xacro (robot description, xacro)
@@ -14,4 +14,10 @@
 				</material>
 			</visual>
+			<collision>
+				<origin xyz="0.006 0.005 ${-mount_collision_padding + (mount_collision_z + 2 * mount_collision_padding) / 2}" rpy="0 0 0" />
+				<geometry>
+					<box size="${mount_collision_x + 2 * mount_collision_padding} ${mount_collision_y + 2 * mount_collision_padding} ${mount_collision_z + 2 * mount_collision_padding}" />
+				</geometry>
+			</collision>
 		</link>
 		<joint name="camera_mount_base_joint" type="fixed">
@@ -21,10 +27,4 @@
 		</joint>
 		<link name="${name}_mount">
-			<collision>
-				<origin xyz="0.006 0.005 ${-mount_collision_padding + (mount_collision_z + 2 * mount_collision_padding) / 2 - 0.0145}" rpy="0 0 0" />
-				<geometry>
-					<box size="${mount_collision_x + 2 * mount_collision_padding} ${mount_collision_y + 2 * mount_collision_padding} ${mount_collision_z + 2 * mount_collision_padding}" />
-				</geometry>
-			</collision>
 		</link>
 		<joint name="${name}_mount_top" type="fixed">

Commit message: Increased camera mount collision box to account for camera cable

File: src/robot_description/urdf/rgbd_camera/mounted_d435i.urdf.xacro (robot description, xacro)
@@ -15,7 +15,7 @@
 			</visual>
 			<collision>
-				<origin xyz="0.006 0.005 ${-mount_collision_padding + (mount_collision_z + 2 * mount_collision_padding) / 2}" rpy="0 0 0" />
+				<origin xyz="0.006 -0.0075 ${-mount_collision_padding + (mount_collision_z + 2 * mount_collision_padding) / 2}" rpy="0 0 0" />
 				<geometry>
-					<box size="${mount_collision_x + 2 * mount_collision_padding} ${mount_collision_y + 2 * mount_collision_padding} ${mount_collision_z + 2 * mount_collision_padding}" />
+					<box size="${mount_collision_x + 2 * mount_collision_padding} ${mount_collision_y + 2 * mount_collision_padding + 0.025} ${mount_collision_z + 2 * mount_collision_padding}" />
 				</geometry>
 			</collision>
