Commit message: Organised the meshes and URDF files

File: src/robot_description/urdf/adaptive_gripper/gripper_with_camera.urdf.xacro (robot description, xacro)
@@ -1,6 +1,6 @@
 <?xml version="1.0"?>
 <robot name="gripper_with_camera" xmlns:xacro="http://www.ros.org/wiki/xacro">
-  <xacro:include filename="$(find robot_description)/urdf/adaptive_gripper.urdf.xacro"/>
-  <xacro:include filename="$(find robot_description)/urdf/mounted_d435i.urdf.xacro"/>
+  <xacro:include filename="$(find robot_description)/urdf/adaptive_gripper/adaptive_gripper.urdf.xacro"/>
+  <xacro:include filename="$(find robot_description)/urdf/rgbd_camera/mounted_d435i.urdf.xacro"/>
   <xacro:macro name="gripper_with_camera" params="parent *origin name:=camera use_nominal_extrinsics:=false">
     <xacro:adaptive_gripper parent="${parent}" prefix="">

File: src/robot_description/urdf/mycobot_280pi/mycobot_280pi.urdf.xacro (robot description, xacro)
@@ -12,5 +12,5 @@
     <xacro:property name="use_gripper_enabled" value="$(arg use_gripper)"/>
     <xacro:property name="use_camera_enabled" value="$(arg use_camera)"/>
-    <xacro:include filename="$(find robot_description)/urdf/mycobot_280pi_arm.urdf.xacro"/>
+    <xacro:include filename="$(find robot_description)/urdf/mycobot_280pi/mycobot_280pi_arm.urdf.xacro"/>
     <link name="$(arg prefix)base_link"/>
     <xacro:mycobot_280pi_arm
@@ -31,5 +31,5 @@
         <xacro:property name="current_gripper" value="$(arg gripper_type)"/>
         <xacro:if value="${current_gripper == 'adaptive_gripper'}">
-            <xacro:include filename="$(find robot_description)/urdf/adaptive_gripper.urdf.xacro"/>
+            <xacro:include filename="$(find robot_description)/urdf/adaptive_gripper/adaptive_gripper.urdf.xacro"/>
             <xacro:adaptive_gripper
                 parent="$(arg flange_link)"
@@ -40,5 +40,5 @@
     </xacro:if>
     <xacro:if value="${use_camera_enabled and not use_gripper_enabled}">
-      <xacro:include filename="$(find robot_description)/urdf/gripper_with_camera.urdf.xacro"/>
+      <xacro:include filename="$(find robot_description)/urdf/adaptive_gripper/gripper_with_camera.urdf.xacro"/>
       <xacro:gripper_with_camera parent="$(arg flange_link)" use_nominal_extrinsics="$(arg use_nominal_extrinsics)">
         <origin xyz="0 0 0.034" rpy="1.579 0 0.785398"/>

File: src/robot_description/urdf/rgbd_camera/_d435.urdf.xacro (robot description, xacro)
@@ -21,6 +21,6 @@
 <robot name="sensor_d435" xmlns:xacro="http://ros.org/wiki/xacro">
   <!-- Includes -->
-  <xacro:include filename="$(find robot_description)/urdf/_materials.urdf.xacro" />
-  <xacro:include filename="$(find robot_description)/urdf/_usb_plug.urdf.xacro" />
+  <xacro:include filename="$(find robot_description)/urdf/rgbd_camera/_materials.urdf.xacro" />
+  <xacro:include filename="$(find robot_description)/urdf/rgbd_camera/_usb_plug.urdf.xacro" />
   <xacro:macro name="sensor_d435" params="parent *origin name:=camera use_nominal_extrinsics:=false add_plug:=false use_mesh:=true">
     <xacro:property name="M_PI" value="3.1415926535897931" />

File: src/robot_description/urdf/rgbd_camera/_d435i.urdf.xacro (robot description, xacro)
@@ -20,6 +20,6 @@
 -->
 <robot name="sensor_d435i" xmlns:xacro="http://ros.org/wiki/xacro">
-  <xacro:include filename="$(find robot_description)/urdf/_d435.urdf.xacro"/>
-  <xacro:include filename="$(find robot_description)/urdf/_d435i_imu_modules.urdf.xacro"/>
+  <xacro:include filename="$(find robot_description)/urdf/rgbd_camera/_d435.urdf.xacro"/>
+  <xacro:include filename="$(find robot_description)/urdf/rgbd_camera/_d435i_imu_modules.urdf.xacro"/>
   <xacro:macro name="sensor_d435i" params="parent *origin name:=camera use_nominal_extrinsics:=false">
     <xacro:sensor_d435 parent="${parent}" name="${name}" use_nominal_extrinsics="${use_nominal_extrinsics}">

File: src/robot_description/urdf/rgbd_camera/_usb_plug.urdf.xacro (robot description, xacro)
@@ -33,5 +33,5 @@
         <geometry>
           <!--box size="0.044850 0.008 0.0185" /-->
-          <mesh filename="package://robot_description/meshes/plug.stl" />
+          <mesh filename="package://robot_description/meshes/rgbd_camera/plug.stl" />
         </geometry>
         <material name="plastic"/>
@@ -41,5 +41,5 @@
         <geometry>
           <!--box size="0.044850 0.008 0.0185" /-->
-          <mesh filename="package://robot_description/meshes/plug_collision.stl" />
+          <mesh filename="package://robot_description/meshes/rgbd_camera/plug_collision.stl" />
         </geometry>
       </collision>

File: src/robot_description/urdf/rgbd_camera/mounted_d435i.urdf.xacro (robot description, xacro)
@@ -8,5 +8,5 @@
 				<origin xyz="0 0 0" rpy="0 0 0" />
 				<geometry>
-					<mesh filename="file://$(find robot_description)/meshes/camera_mount.stl" scale="${mount_mesh_scale} ${mount_mesh_scale} ${mount_mesh_scale}" />
+					<mesh filename="file://$(find robot_description)/meshes/rgbd_camera/camera_mount.stl" scale="${mount_mesh_scale} ${mount_mesh_scale} ${mount_mesh_scale}" />
 				</geometry>
 				<material name="mount_gray">

File: src/robot_description/urdf/view/view_adaptive_gripper.urdf.xacro (robot description, xacro)
@@ -1,5 +1,5 @@
 <?xml version="1.0"?>
 <robot name="adaptive_gripper" xmlns:xacro="http://www.ros.org/wiki/xacro">
-  <xacro:include filename="$(find robot_description)/urdf/adaptive_gripper.urdf.xacro"/>
+  <xacro:include filename="$(find robot_description)/urdf/adaptive_gripper/adaptive_gripper.urdf.xacro"/>
   <link name="base_link" />
   <xacro:adaptive_gripper parent="base_link" prefix="">

File: src/robot_description/urdf/view/view_d435i_camera.urdf.xacro (robot description, xacro)
@@ -2,5 +2,5 @@
 <robot name="d435i" xmlns:xacro="http://www.ros.org/wiki/xacro">
   <xacro:arg name="use_nominal_extrinsics" default="false" />
-  <xacro:include filename="$(find robot_description)/urdf/_d435i.urdf.xacro"/>
+  <xacro:include filename="$(find robot_description)/urdf/rgbd_camera/_d435i.urdf.xacro"/>
   <link name="base_link" />
   <xacro:sensor_d435i parent="base_link" use_nominal_extrinsics="$(arg use_nominal_extrinsics)">

File: src/robot_description/urdf/view/view_gripper_with_camera.urdf.xacro (robot description, xacro)
@@ -2,5 +2,5 @@
 <robot name="gripper_with_camera" xmlns:xacro="http://www.ros.org/wiki/xacro">
   <xacro:arg name="use_nominal_extrinsics" default="false" />
-  <xacro:include filename="$(find robot_description)/urdf/gripper_with_camera.urdf.xacro"/>
+  <xacro:include filename="$(find robot_description)/urdf/adaptive_gripper/agripper_with_camera.urdf.xacro"/>
   <link name="base_link" />
   <xacro:gripper_with_camera parent="base_link" name="camera" use_nominal_extrinsics="$(arg use_nominal_extrinsics)">

File: src/robot_description/urdf/view/view_mounted_d435i.urdf.xacro (robot description, xacro)
@@ -2,5 +2,5 @@
 <robot name="mounted_d435i" xmlns:xacro="http://www.ros.org/wiki/xacro">
   <xacro:arg name="use_nominal_extrinsics" default="false" />
-  <xacro:include filename="$(find robot_description)/urdf/mounted_d435i.urdf.xacro"/>
+  <xacro:include filename="$(find robot_description)/urdf/rgbd_camera/mounted_d435i.urdf.xacro"/>
   <link name="base_link" />
   <xacro:mounted_d435i parent="base_link" name="camera" use_nominal_extrinsics="$(arg use_nominal_extrinsics)">

File: src/robot_description/urdf/view/view_mycobot_280pi.urdf.xacro (robot description, xacro)
@@ -1,4 +1,4 @@
 <?xml version="1.0"?>
 <robot name="mycobot_280pi" xmlns:xacro="http://www.ros.org/wiki/xacro">
-  <xacro:include filename="$(find robot_description)/urdf/mycobot_280pi.urdf.xacro"/>
+  <xacro:include filename="$(find robot_description)/urdf/mycobot_280pi/mycobot_280pi.urdf.xacro"/>
 </robot>

File: src/robot_description/urdf/view/view_mycobot_280pi_arm.urdf.xacro (robot description, xacro)
@@ -1,5 +1,5 @@
 <?xml version="1.0"?>
 <robot name="mycobot_280pi" xmlns:xacro="http://www.ros.org/wiki/xacro">
-  <xacro:include filename="$(find robot_description)/urdf/mycobot_280pi_arm.urdf.xacro"/>
+  <xacro:include filename="$(find robot_description)/urdf/mycobot_280pi/mycobot_280pi_arm.urdf.xacro"/>
   <link name="base_link" />
   <xacro:mycobot_280pi_arm base_link="base_link" flange_link="link6_flange" prefix="">

Commit message: Rename URDF

File: src/robot_description/urdf/adaptive_gripper/gripper_with_camera.urdf.xacro (robot description, xacro)
@@ -2,12 +2,12 @@
 <robot name="gripper_with_camera" xmlns:xacro="http://www.ros.org/wiki/xacro">
   <xacro:include filename="$(find robot_description)/urdf/adaptive_gripper/adaptive_gripper.urdf.xacro"/>
-  <xacro:include filename="$(find robot_description)/urdf/rgbd_camera/mounted_d435i.urdf.xacro"/>
+  <xacro:include filename="$(find robot_description)/urdf/rgbd_camera/d435i_mounted.urdf.xacro"/>
   <xacro:macro name="gripper_with_camera" params="parent *origin name:=camera use_nominal_extrinsics:=false">
     <xacro:adaptive_gripper parent="${parent}" prefix="">
       <xacro:insert_block name="origin"/>
     </xacro:adaptive_gripper>
-    <xacro:mounted_d435i parent="gripper_mount" name="${name}" use_nominal_extrinsics="${use_nominal_extrinsics}">
+    <xacro:d435i_mounted parent="gripper_mount" name="${name}" use_nominal_extrinsics="${use_nominal_extrinsics}">
       <origin xyz="0 0 0" rpy="3.141592653589793 0 1.5707963267948966" />
-    </xacro:mounted_d435i>
+    </xacro:d435i_mounted>
   </xacro:macro>
 </robot>

File: src/robot_description/urdf/rgbd_camera/d435i_mounted.urdf.xacro (robot description, xacro)
@@ -1,6 +1,6 @@
 <?xml version="1.0"?>
-<robot name="mounted_d435i" xmlns:xacro="http://www.ros.org/wiki/xacro">
+<robot name="d435i_mounted" xmlns:xacro="http://www.ros.org/wiki/xacro">
 	<xacro:include filename="$(find robot_description)/urdf/rgbd_camera/_d435i.urdf.xacro"/>
-	<xacro:macro name="mounted_d435i" params="parent *origin name:=camera use_nominal_extrinsics:=false mount_mesh_scale:=1.0 mount_mesh_x:=0.04073 mount_mesh_y:=0.1082 mount_mesh_z:=0.05081 mount_collision_x:=0.04073 mount_collision_y:=0.1082 mount_collision_z:=0.05081">
+	<xacro:macro name="d435i_mounted" params="parent *origin name:=camera use_nominal_extrinsics:=false mount_mesh_scale:=1.0 mount_mesh_x:=0.04073 mount_mesh_y:=0.1082 mount_mesh_z:=0.05081 mount_collision_x:=0.04073 mount_collision_y:=0.1082 mount_collision_z:=0.05081">
 		<xacro:property name="mount_collision_padding" value="0.005" />
 		<link name="camera_mount_base">

Commit message: Added namespacing to cobot urdf

File: src/robot_description/urdf/adaptive_gripper/gripper_with_camera.urdf.xacro (robot description, xacro)
@@ -3,9 +3,9 @@
   <xacro:include filename="$(find robot_description)/urdf/adaptive_gripper/adaptive_gripper.urdf.xacro"/>
   <xacro:include filename="$(find robot_description)/urdf/rgbd_camera/d435i_mounted.urdf.xacro"/>
-  <xacro:macro name="gripper_with_camera" params="parent *origin name:=camera use_nominal_extrinsics:=false">
-    <xacro:adaptive_gripper parent="${parent}" prefix="">
+  <xacro:macro name="gripper_with_camera" params="parent *origin name:=camera prefix:='' use_nominal_extrinsics:=false">
+    <xacro:adaptive_gripper parent="${parent}" prefix="${prefix}">
       <xacro:insert_block name="origin"/>
     </xacro:adaptive_gripper>
-    <xacro:d435i_mounted parent="gripper_mount" name="${name}" use_nominal_extrinsics="${use_nominal_extrinsics}">
+    <xacro:d435i_mounted parent="${prefix}gripper_mount" name="${name}" prefix="${prefix}" use_nominal_extrinsics="${use_nominal_extrinsics}">
       <origin xyz="0 0 0" rpy="3.141592653589793 0 1.5707963267948966" />
     </xacro:d435i_mounted>

File: src/robot_description/urdf/mycobot_280pi/mycobot_280pi.urdf.xacro (robot description, xacro)
@@ -3,26 +3,31 @@
     <xacro:arg name="robot_name" default="mycobot_280pi"/>
     <xacro:arg name="add_world" default="true"/>
+    <xacro:arg name="cobot_ns" default="cobot"/>
     <xacro:arg name="flange_link" default="link6_flange"/>
-    <xacro:arg name="prefix" default=""/>
     <xacro:arg name="use_nominal_extrinsics" default="true"/>
     <xacro:arg name="use_gazebo" default="false"/>
+    <!-- Compute prefix from cobot_ns, same as leo -->
+    <xacro:property name="prefix" value=""/>
+    <xacro:if value="${'$(arg cobot_ns)' != '' and '$(arg cobot_ns)' != '/'}">
+      <xacro:property name="prefix" value="$(arg cobot_ns)/"/>
+    </xacro:if>
     <xacro:include filename="$(find robot_description)/urdf/mycobot_280pi/mycobot_280pi_arm.urdf.xacro"/>
-    <link name="$(arg prefix)base_link"/>
+    <link name="${prefix}base_link"/>
     <xacro:mycobot_280pi_arm
       base_link="base_link"
       flange_link="$(arg flange_link)"
-      prefix="$(arg prefix)">
+      prefix="${prefix}">
       <origin xyz="0 0 0" rpy="0 0 0"/>
     </xacro:mycobot_280pi_arm>
     <xacro:if value="$(arg add_world)">
       <link name="world"/>
-      <joint name="$(arg prefix)virtual_joint" type="fixed">
+      <joint name="${prefix}virtual_joint" type="fixed">
           <parent link="world"/>
-          <child link="$(arg prefix)base_link"/>
+          <child link="${prefix}base_link"/>
           <origin xyz="0 0 0" rpy="0 0 0"/>
       </joint>
     </xacro:if>
     <xacro:include filename="$(find robot_description)/urdf/adaptive_gripper/gripper_with_camera.urdf.xacro"/>
-    <xacro:gripper_with_camera parent="$(arg flange_link)" name="camera" use_nominal_extrinsics="$(arg use_nominal_extrinsics)">
+    <xacro:gripper_with_camera parent="$(arg flange_link)" prefix="${prefix}" name="${prefix}camera" use_nominal_extrinsics="$(arg use_nominal_extrinsics)">
       <origin xyz="0 0 0.034" rpy="1.579 0 0.785398"/>
     </xacro:gripper_with_camera>
@@ -33,5 +38,5 @@
     <xacro:include filename="$(find robot_description)/urdf/control/mycobot_280_ros2_control.urdf.xacro" />
     <xacro:mycobot_ros2_control
-      prefix="$(arg prefix)"
+      prefix="${prefix}"
       flange_link="$(arg flange_link)"
       use_gazebo="$(arg use_gazebo)"/>

File: src/robot_description/urdf/rgbd_camera/d435i_mounted.urdf.xacro (robot description, xacro)
@@ -2,7 +2,7 @@
 <robot name="d435i_mounted" xmlns:xacro="http://www.ros.org/wiki/xacro">
 	<xacro:include filename="$(find robot_description)/urdf/rgbd_camera/_d435i.urdf.xacro"/>
-	<xacro:macro name="d435i_mounted" params="parent *origin name:=camera use_nominal_extrinsics:=false mount_mesh_scale:=1.0 mount_mesh_x:=0.04073 mount_mesh_y:=0.1082 mount_mesh_z:=0.05081 mount_collision_x:=0.04073 mount_collision_y:=0.1082 mount_collision_z:=0.05081">
+	<xacro:macro name="d435i_mounted" params="parent *origin name:=camera prefix:='' use_nominal_extrinsics:=false mount_mesh_scale:=1.0 mount_mesh_x:=0.04073 mount_mesh_y:=0.1082 mount_mesh_z:=0.05081 mount_collision_x:=0.04073 mount_collision_y:=0.1082 mount_collision_z:=0.05081">
 		<xacro:property name="mount_collision_padding" value="0.005" />
-		<link name="camera_mount_base">
+		<link name="${prefix}camera_mount_base">
 			<visual>
 				<origin xyz="0 0 0" rpy="0 0 0" />
@@ -21,17 +21,17 @@
 			</collision>
 		</link>
-		<joint name="camera_mount_base_joint" type="fixed">
+		<joint name="${prefix}camera_mount_base_joint" type="fixed">
 			<xacro:insert_block name="origin" />
 			<parent link="${parent}" />
-			<child link="camera_mount_base" />
+			<child link="${prefix}camera_mount_base" />
 		</joint>
-		<link name="${name}_mount">
+		<link name="${prefix}${name}_mount">
 		</link>
-		<joint name="${name}_mount_top" type="fixed">
-			<parent link="camera_mount_base" />
-			<child link="${name}_mount" />
+		<joint name="${prefix}${name}_mount_top" type="fixed">
+			<parent link="${prefix}camera_mount_base" />
+			<child link="${prefix}${name}_mount" />
             <origin xyz="0 0 0.0145" rpy="0 0 0" />
 		</joint>
-		<xacro:sensor_d435i parent="${name}_mount" name="${name}" use_nominal_extrinsics="${use_nominal_extrinsics}">
+		<xacro:sensor_d435i parent="${prefix}${name}_mount" name="${prefix}${name}" use_nominal_extrinsics="${use_nominal_extrinsics}">
 			<origin xyz="0.006 0 0" rpy="0 0 0" /> // Not sure of exact offset, delta x from central hole on camera mount to center of camera screw mount
 		</xacro:sensor_d435i>
