Commit message: Removed unecessary use_camera and use_gripper args

File: src/robot_description/urdf/mycobot_280pi/mycobot_280pi.urdf.xacro (robot description, xacro)
@@ -4,12 +4,7 @@
     <xacro:arg name="add_world" default="true"/>
     <xacro:arg name="flange_link" default="link6_flange"/>
-    <xacro:arg name="gripper_type" default="adaptive_gripper"/>
     <xacro:arg name="prefix" default=""/>
-    <xacro:arg name="use_camera" default="true"/>
     <xacro:arg name="use_nominal_extrinsics" default="true"/>
     <xacro:arg name="use_gazebo" default="false"/>
-    <xacro:arg name="use_gripper" default="false"/>
-    <xacro:property name="use_gripper_enabled" value="$(arg use_gripper)"/>
-    <xacro:property name="use_camera_enabled" value="$(arg use_camera)"/>
     <xacro:include filename="$(find robot_description)/urdf/mycobot_280pi/mycobot_280pi_arm.urdf.xacro"/>
     <link name="$(arg prefix)base_link"/>
@@ -28,21 +23,8 @@
       </joint>
     </xacro:if>
-    <xacro:if value="${use_gripper_enabled and not use_camera_enabled}">
-        <xacro:property name="current_gripper" value="$(arg gripper_type)"/>
-        <xacro:if value="${current_gripper == 'adaptive_gripper'}">
-            <xacro:include filename="$(find robot_description)/urdf/adaptive_gripper/adaptive_gripper.urdf.xacro"/>
-            <xacro:adaptive_gripper
-                parent="$(arg flange_link)"
-                prefix="$(arg prefix)">
-                <origin xyz="0 0 0.034" rpy="1.579 0 0.785398"/>
-            </xacro:adaptive_gripper>
-        </xacro:if>
-    </xacro:if>
-    <xacro:if value="${use_camera_enabled and not use_gripper_enabled}">
-      <xacro:include filename="$(find robot_description)/urdf/adaptive_gripper/gripper_with_camera.urdf.xacro"/>
-      <xacro:gripper_with_camera parent="$(arg flange_link)" use_nominal_extrinsics="$(arg use_nominal_extrinsics)">
-        <origin xyz="0 0 0.034" rpy="1.579 0 0.785398"/>
-      </xacro:gripper_with_camera>
-    </xacro:if>
+    <xacro:include filename="$(find robot_description)/urdf/adaptive_gripper/gripper_with_camera.urdf.xacro"/>
+    <xacro:gripper_with_camera parent="$(arg flange_link)" name="camera" use_nominal_extrinsics="$(arg use_nominal_extrinsics)">
+      <origin xyz="0 0 0.034" rpy="1.579 0 0.785398"/>
+    </xacro:gripper_with_camera>
     <xacro:include filename="$(find robot_description)/urdf/control/gazebo_sim_ros2_control.urdf.xacro" />
     <xacro:load_gazebo_sim_ros2_control_plugin
