Commit message: Fixed cobot link1 orientation

File: src/robot_description/urdf/mycobot_280pi/mycobot_280pi_arm.urdf.xacro (robot description, xacro)
@@ -40,6 +40,6 @@
           <mesh filename="file://$(find robot_description)/meshes/mycobot_280_pi/link1.dae"/>
         </geometry>
-        <origin xyz="0.0 0 0" rpy="0 0 ${-pi/2}"/>
-      </visual>
+        <origin xyz="0.0 0 0" rpy="0 0 ${-pi}"/>
+      </visual>-
       <collision>
         <geometry>
