Commit message: Blender file folder added, urdf restructured and updated (still in progress)

File: src/leo_simulator-ros2/leo_full_description/launch/leo_sim_1.urdf.xacro (robot description, xacro)
@@ -6,6 +6,9 @@
   <xacro:arg name="mecanum_wheels" default="false"/>
   <xacro:include filename="$(find leo_description)/urdf/macros.xacro"/>
+  <xacro:include filename="$(find leo_full_description)/urdf/mounting_plate.urdf.xacro"/>
   <xacro:leo_sim robot_ns="$(arg robot_ns)"
                  fixed="$(arg fixed)"
                  mecanum_wheels="$(arg mecanum_wheels)"/>
+  <xacro:mounting_plate parent="base_link" prefix="$(arg robot_ns)">
+    <origin xyz="0.06 0.02 0" rpy="0 0 0"/> </xacro:mounting_plate>
 </robot>

Commit message: urdf models working, not positioned correctly, lidar setup still required

File: src/leo_simulator-ros2/leo_full_description/launch/leo_sim_1.urdf.xacro (robot description, xacro)
@@ -7,8 +7,11 @@
   <xacro:include filename="$(find leo_description)/urdf/macros.xacro"/>
   <xacro:include filename="$(find leo_full_description)/urdf/mounting_plate.urdf.xacro"/>
+  <xacro:include filename="$(find leo_full_description)/urdf/nuc_assemb.urdf.xacro"/>
   <xacro:leo_sim robot_ns="$(arg robot_ns)"
                  fixed="$(arg fixed)"
                  mecanum_wheels="$(arg mecanum_wheels)"/>
-  <xacro:mounting_plate parent="base_link" prefix="$(arg robot_ns)">
+  <xacro:mounting_plate parent="$(arg robot_ns)/base_link" prefix="$(arg robot_ns)/">
     <origin xyz="0.06 0.02 0" rpy="0 0 0"/> </xacro:mounting_plate>
+  <xacro:nuc_assemb parent="$(arg robot_ns)/rocker_R_link" prefix="$(arg robot_ns)/">
+    <origin xyz="-0.15 0.02 0" rpy="0 0 0"/> </xacro:nuc_assemb>
 </robot>

File: src/leo_simulator-ros2/leo_full_description/urdf/mounting_plate.urdf.xacro (robot description, xacro)
@@ -1,5 +1,5 @@
 <?xml version="1.0"?>
 <robot xmlns:xacro="http://ros.org/wiki/xacro">
-  <xacro:macro name="mounting_plate" params="parent prefix *origin">
+  <xacro:macro name="mounting_plate" params="parent prefix *origin mount_mesh_scale:=1.0">
     <joint name="${prefix}mounting_plate_joint" type="fixed">
       <xacro:insert_block name="origin" />
@@ -10,10 +10,10 @@
       <visual>
         <geometry>
-          <mesh filename="package://leo_full_description/meshes/mounting_plate.dae" scale="${mount_mesh_scale} ${mount_mesh_scale} ${mount_mesh_scale}" />
+          <mesh filename="$(find leo_full_description)/meshes/mounting_plate_assemb.dae" scale="${mount_mesh_scale} ${mount_mesh_scale} ${mount_mesh_scale}" />
         </geometry>
       </visual>
       <collision>
         <geometry>
-          <mesh filename="package://leo_full_description/meshes/mounting_plate.dae" scale="${mount_mesh_scale} ${mount_mesh_scale} ${mount_mesh_scale}" />
+          <mesh filename="$(find leo_full_description)/meshes/mounting_plate_assemb.dae" scale="${mount_mesh_scale} ${mount_mesh_scale} ${mount_mesh_scale}" />
         </geometry>
       </collision>

Commit message: Working Rviz configuration

File: src/leo_simulator-ros2/leo_full_description/launch/leo_sim_1.urdf.xacro (robot description, xacro)
@@ -8,10 +8,16 @@
   <xacro:include filename="$(find leo_full_description)/urdf/mounting_plate.urdf.xacro"/>
   <xacro:include filename="$(find leo_full_description)/urdf/nuc_assemb.urdf.xacro"/>
+  <xacro:include filename="$(find leo_full_description)/urdf/lidar.urdf.xacro"/>
+  <xacro:include filename="$(find leo_full_description)/urdf/lidar_mount.urdf.xacro"/>
   <xacro:leo_sim robot_ns="$(arg robot_ns)"
                  fixed="$(arg fixed)"
                  mecanum_wheels="$(arg mecanum_wheels)"/>
   <xacro:mounting_plate parent="$(arg robot_ns)/base_link" prefix="$(arg robot_ns)/">
-    <origin xyz="0.06 0.02 0" rpy="0 0 0"/> </xacro:mounting_plate>
+    <origin xyz="0.0295 0.00458 0.02525" rpy="0 0 1.570796327"/> </xacro:mounting_plate>
   <xacro:nuc_assemb parent="$(arg robot_ns)/rocker_R_link" prefix="$(arg robot_ns)/">
-    <origin xyz="-0.15 0.02 0" rpy="0 0 0"/> </xacro:nuc_assemb>
+    <origin xyz="-0.10644 -0.02816 0.0254" rpy="0 0 1.570796327"/> </xacro:nuc_assemb>
+  <xacro:lidar parent="$(arg robot_ns)/base_link" prefix="$(arg robot_ns)/">
+    <origin xyz="0.09 0.009 0.023" rpy="0 0 0"/> </xacro:lidar>
+  <xacro:lidar_mount parent="$(arg robot_ns)/base_link" prefix="$(arg robot_ns)/">
+    <origin xyz="0.0775 0.009 0.0025" rpy="0 0 3.141592654"/> </xacro:lidar_mount>
 </robot>

File: src/leo_simulator-ros2/leo_full_description/urdf/mounting_plate.urdf.xacro (robot description, xacro)
@@ -10,10 +10,10 @@
       <visual>
         <geometry>
-          <mesh filename="$(find leo_full_description)/meshes/mounting_plate_assemb.dae" scale="${mount_mesh_scale} ${mount_mesh_scale} ${mount_mesh_scale}" />
+          <mesh filename="package://leo_full_description/meshes/mounting_plate_assemb.dae" scale="${mount_mesh_scale} ${mount_mesh_scale} ${mount_mesh_scale}" />
         </geometry>
       </visual>
       <collision>
         <geometry>
-          <mesh filename="$(find leo_full_description)/meshes/mounting_plate_assemb.dae" scale="${mount_mesh_scale} ${mount_mesh_scale} ${mount_mesh_scale}" />
+          <mesh filename="package://leo_full_description/meshes/mounting_plate_assemb.dae" scale="${mount_mesh_scale} ${mount_mesh_scale} ${mount_mesh_scale}" />
         </geometry>
       </collision>

File: src/leo_simulator-ros2/leo_full_description/urdf/nuc_assemb.urdf.xacro (robot description, xacro)
@@ -10,10 +10,10 @@
       <visual>
         <geometry>
-          <mesh filename="$(find leo_full_description)/meshes/nuc_assmb.dae" scale="${mount_mesh_scale} ${mount_mesh_scale} ${mount_mesh_scale}" />
+          <mesh filename="package://leo_full_description/meshes/nuc_assmb.dae" scale="${mount_mesh_scale} ${mount_mesh_scale} ${mount_mesh_scale}" />
         </geometry>
       </visual>
       <collision>
         <geometry>
-          <mesh filename="$(find leo_full_description)/meshes/nuc_assmb.dae" scale="${mount_mesh_scale} ${mount_mesh_scale} ${mount_mesh_scale}" />
+          <mesh filename="package://leo_full_description/meshes/nuc_assmb.dae" scale="${mount_mesh_scale} ${mount_mesh_scale} ${mount_mesh_scale}" />
         </geometry>
       </collision>
