Commit message: Added mounting plate link

File: src/leo_simulator-ros2/leo_full_description/urdf/mounting_plate.urdf.xacro (robot description, xacro)
@@ -19,4 +19,12 @@
       </collision>
     </link>
+    <link name="${prefix}cobot_mount_link">
+    </link>
+    <joint name="${prefix}cobot_mount" type="fixed">
+      <xacro:insert_block name="origin" />
+      <parent link="${prefix}mounting_plate_link"/>
+      <child link="${prefix}cobot_mount_link"/>
+      <origin xyz="0.0 0.0 0.03" rpy="0 0 0"/>
+    </joint>
   </xacro:macro>
 </robot>

Commit message: Link added for attaching the cobot to the top of the mounting plate

File: src/leo_simulator-ros2/leo_full_description/urdf/mounting_plate.urdf.xacro (robot description, xacro)
@@ -19,12 +19,11 @@
       </collision>
     </link>
-    <link name="${prefix}cobot_mount_link">
-    </link>
-    <joint name="${prefix}cobot_mount" type="fixed">
-      <xacro:insert_block name="origin" />
-      <parent link="${prefix}mounting_plate_link"/>
-      <child link="${prefix}cobot_mount_link"/>
-      <origin xyz="0.0 0.0 0.03" rpy="0 0 0"/>
-    </joint>
+    <link name="${prefix}cobot_manipulator_mount_link">
+		</link>
+		<joint name="$${prefix}cobot_manipulator_mount" type="fixed">
+			<parent link="${prefix}mounting_plate_link" />
+			<child link="${prefix}cobot_manipulator_mount_link" />
+            <origin xyz="0.004425 -0.001 0.03475" rpy="0 0 0" />
+		</joint>
   </xacro:macro>
 </robot>

Commit message: Remove double $

File: src/leo_simulator-ros2/leo_full_description/urdf/mounting_plate.urdf.xacro (robot description, xacro)
@@ -21,5 +21,5 @@
     <link name="${prefix}cobot_manipulator_mount_link">
 		</link>
-		<joint name="$${prefix}cobot_manipulator_mount" type="fixed">
+		<joint name="${prefix}cobot_manipulator_mount" type="fixed">
 			<parent link="${prefix}mounting_plate_link" />
 			<child link="${prefix}cobot_manipulator_mount_link" />
