Commit message: Models working in both rviz and gazebo

File: src/leo_simulator-ros2/leo_full_description/urdf/lidar.urdf.xacro (robot description, xacro)
@@ -10,10 +10,10 @@
       <visual>
         <geometry>
-          <mesh filename="package://leo_full_description/meshes/lidar.dae" scale="${mount_mesh_scale} ${mount_mesh_scale} ${mount_mesh_scale}" />
+          <mesh filename="file://$(find leo_full_description)/meshes/lidar.dae" scale="${mount_mesh_scale} ${mount_mesh_scale} ${mount_mesh_scale}" />
         </geometry>
       </visual>
       <collision>
         <geometry>
-          <mesh filename="package://leo_full_description/meshes/lidar.dae" scale="${mount_mesh_scale} ${mount_mesh_scale} ${mount_mesh_scale}" />
+          <mesh filename="file://$(find leo_full_description)/meshes/lidar.dae" scale="${mount_mesh_scale} ${mount_mesh_scale} ${mount_mesh_scale}" />
         </geometry>
       </collision>

File: src/leo_simulator-ros2/leo_full_description/urdf/lidar_mount.urdf.xacro (robot description, xacro)
@@ -10,10 +10,10 @@
       <visual>
         <geometry>
-          <mesh filename="package://leo_full_description/meshes/lidar_mount.dae" scale="${mount_mesh_scale} ${mount_mesh_scale} ${mount_mesh_scale}" />
+          <mesh filename="file://$(find leo_full_description)/meshes/lidar_mount.dae" scale="${mount_mesh_scale} ${mount_mesh_scale} ${mount_mesh_scale}" />
         </geometry>
       </visual>
       <collision>
         <geometry>
-          <mesh filename="package://leo_full_description/meshes/lidar_mount.dae" scale="${mount_mesh_scale} ${mount_mesh_scale} ${mount_mesh_scale}" />
+          <mesh filename="file://$(find leo_full_description)/meshes/lidar_mount.dae" scale="${mount_mesh_scale} ${mount_mesh_scale} ${mount_mesh_scale}" />
         </geometry>
       </collision>

File: src/leo_simulator-ros2/leo_full_description/urdf/mounting_plate.urdf.xacro (robot description, xacro)
@@ -10,10 +10,10 @@
       <visual>
         <geometry>
-          <mesh filename="package://leo_full_description/meshes/mounting_plate_assemb.dae" scale="${mount_mesh_scale} ${mount_mesh_scale} ${mount_mesh_scale}" />
+          <mesh filename="file://$(find leo_full_description)/meshes/mounting_plate_assemb.dae" scale="${mount_mesh_scale} ${mount_mesh_scale} ${mount_mesh_scale}" />
         </geometry>
       </visual>
       <collision>
         <geometry>
-          <mesh filename="package://leo_full_description/meshes/mounting_plate_assemb.dae" scale="${mount_mesh_scale} ${mount_mesh_scale} ${mount_mesh_scale}" />
+          <mesh filename="file://$(find leo_full_description)/meshes/mounting_plate_assemb.dae" scale="${mount_mesh_scale} ${mount_mesh_scale} ${mount_mesh_scale}" />
         </geometry>
       </collision>

File: src/leo_simulator-ros2/leo_full_description/urdf/nuc_assemb.urdf.xacro (robot description, xacro)
@@ -10,10 +10,10 @@
       <visual>
         <geometry>
-          <mesh filename="package://leo_full_description/meshes/nuc_assmb.dae" scale="${mount_mesh_scale} ${mount_mesh_scale} ${mount_mesh_scale}" />
+          <mesh filename="file://$(find leo_full_description)/meshes/nuc_assmb.dae" scale="${mount_mesh_scale} ${mount_mesh_scale} ${mount_mesh_scale}" />
         </geometry>
       </visual>
       <collision>
         <geometry>
-          <mesh filename="package://leo_full_description/meshes/nuc_assmb.dae" scale="${mount_mesh_scale} ${mount_mesh_scale} ${mount_mesh_scale}" />
+          <mesh filename="file://$(find leo_full_description)/meshes/nuc_assmb.dae" scale="${mount_mesh_scale} ${mount_mesh_scale} ${mount_mesh_scale}" />
         </geometry>
       </collision>

Commit message: lidar sensor added

File: src/leo_simulator-ros2/leo_full_description/urdf/lidar.urdf.xacro (robot description, xacro)
@@ -1,4 +1,4 @@
 <?xml version="1.0"?>
-<robot xmlns:xacro="http://ros.org/wiki/xacro">
+<robot xmlns:xacro="http://www.ros.org/wiki/xacro">
   <xacro:macro name="lidar" params="parent prefix *origin mount_mesh_scale:=1.0">
     <joint name="${prefix}lidar_joint" type="fixed">
@@ -8,4 +8,9 @@
     </joint>
     <link name="${prefix}lidar_link">
+      <inertial>
+        <mass value="0.1"/>
+        <origin xyz="0 0 0" rpy="0 0 0"/>
+        <inertia ixx="1e-6" ixy="0" ixz="0" iyy="1e-6" iyz="0" izz="1e-6"/>
+      </inertial>
       <visual>
         <geometry>
@@ -15,8 +20,38 @@
       <collision>
         <geometry>
-          <mesh filename="file://$(find leo_full_description)/meshes/lidar.dae" scale="${mount_mesh_scale} ${mount_mesh_scale} ${mount_mesh_scale}" />
+          <cylinder radius="0.035" length="0.04"/>
         </geometry>
       </collision>
     </link>
+    <gazebo reference="${prefix}lidar_link">
+      <sensor name="intel_realsense_r200" type="gpu_lidar">
+        <gz_frame_id>${prefix}lidar_link</gz_frame_id>
+        <pose>0 0 0 0 0 0</pose>
+        <always_on>true</always_on>
+        <visualize>true</visualize>
+        <update_rate>10</update_rate>
+        <topic>${prefix}scan</topic>
+        <ray>
+          <scan>
+            <horizontal>
+              <samples>360</samples>
+              <resolution>1</resolution>
+              <min_angle>-3.14159</min_angle>
+              <max_angle>3.14159</max_angle>
+            </horizontal>
+          </scan>
+          <range>
+            <min>0.12</min>
+            <max>12.0</max>
+            <resolution>0.01</resolution>
+          </range>
+          <noise>
+            <type>gaussian</type>
+            <mean>0.0</mean>
+            <stddev>0.01</stddev>
+          </noise>
+        </ray>
+      </sensor>
+    </gazebo>
   </xacro:macro>
 </robot>
